File: Hardware/constellation/magnometer.kicad_sch (KiCad schematic)
At the start: 4 parts, among them U6 MMC5983MA

Commit message: add the hierarchal pins to the imu block
Changed lines of the file:
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@@
 		)
 	)
-	(global_label "MMC_MISO"
+	(hierarchical_label "MMC_INT"
+		(shape input)
+		(at 161.29 95.25 0)
+		(effects
+			(font
+				(size 1.27 1.27)
+			)
+			(justify left)
+		)
+	)
+	(hierarchical_label "MMC_MISO"
 		(shape input)
 		(at 111.76 100.33 180)
-		(fields_autoplaced yes)
 		(effects
 			(font
@@
 			(justify right)
 		)
-		(property "Intersheetrefs" "${INTERSHEET_REFS}"
-			(at 92.7487 100.33 0)
-			(hide yes)
-			(show_name no)
-			(do_not_autoplace no)
-			(effects
-				(font
-					(size 1.27 1.27)
-				)
-				(justify right)
-			)
-		)
 	)
-	(global_label "MMC_SCK"
+	(hierarchical_label "MMC_MOSI"
 		(shape input)
-		(at 111.76 97.79 180)
-		(fields_autoplaced yes)
+		(at 111.76 102.87 180)
 		(effects
 			(font
@@
 			(justify right)
 		)
-		(property "Intersheetrefs" "${INTERSHEET_REFS}"
-			(at 92.7487 97.79 0)
-			(hide yes)
-			(show_name no)
-			(do_not_autoplace no)
-			(effects
-				(font
-					(size 1.27 1.27)
-				)
-				(justify right)
-			)
-		)
 	)
-	(global_label "MMC_CS"
+	(hierarchical_label "MMC_CS"
 		(shape input)
 		(at 111.76 95.25 180)
-		(fields_autoplaced yes)
 		(effects
 			(font
@@
 			(justify right)
 		)
-		(property "Intersheetrefs" "${INTERSHEET_REFS}"
-			(at 92.7487 95.25 0)
-			(hide yes)
-			(show_name no)
-			(do_not_autoplace no)
-			(effects
-				(font
-					(size 1.27 1.27)
-				)
-				(justify right)
-			)
-		)
 	)
-	(global_label "MMC_MOSI"
+	(hierarchical_label "MMC_SCK"
 		(shape input)
-		(at 111.76 102.87 180)
-		(fields_autoplaced yes)
+		(at 111.76 97.79 180)
 		(effects
 			(font
@@
 			(justify right)
 		)
-		(property "Intersheetrefs" "${INTERSHEET_REFS}"
-			(at 92.7487 102.87 0)
-			(hide yes)
-			(show_name no)
-			(do_not_autoplace no)
-			(effects
-				(font
-					(size 1.27 1.27)
-				)
-				(justify right)
-			)
-		)
 	)
-	(global_label "MMC_INT"
-		(shape input)
-		(at 161.29 95.25 0)
-		(fields_autoplaced yes)
-		(effects
-			(font
-				(size 1.27 1.27)
-			)
-			(justify left)
-		)
-		(property "Intersheetrefs" "${INTERSHEET_REFS}"
-			(at 180.3013 95.25 0)
-			(hide yes)
-			(show_name no)
-			(do_not_autoplace no)
-			(effects
-				(font
-					(size 1.27 1.27)
-				)
-				(justify left)
-			)
-		)
-	)
