File: Hardware/constellation/magnometer.kicad_sch (KiCad schematic)
At the start: 4 parts, among them U6 MMC5983MA

Commit message: add lr2021 footprint and comms
Parts:
- removed C8: 10uF, Capacitor_SMD:C_0402_1005Metric, symbol Device:C_Small
- removed C9: 1uF, Capacitor_SMD:C_0402_1005Metric, symbol Device:C_Small
- removed R5: 10K, Resistor_SMD:R_0402_1005Metric_Pad0.72x0.64mm_HandSolder, symbol Device:R_Small
- added C15: 10uF, Capacitor_SMD:C_0402_1005Metric, symbol Device:C_Small
- added C20: 1uF, Capacitor_SMD:C_0402_1005Metric, symbol Device:C_Small
- added R13: 10K, Resistor_SMD:R_0402_1005Metric_Pad0.72x0.64mm_HandSolder, symbol Device:R_Small
Connections:
- net GND: now also C15.2, C20.2
- net MMC_CS: now also R13.2
- net VDD: now also C20.1, R13.1
- net at U6.10 (CAP): now also C15.1
- no-connect marks 0 -> 1
Other:
- title: Magnetometer -> Barometric Unit Array
