File: Hardware/constellation/gnss.kicad_sch (KiCad schematic)
At the start: 11 parts, among them J2 U.FL, Q3 BSS138, Q4 BSS83P, U13 MIA-M10C, Y3 32.768 KHZ

Commit message: add lr2021 footprint and comms
Parts:
- renumbered C22 to C12, J2 to J1, L2 to L1, Q3 to Q1, Q4 to Q2, R2 to R10, R16 to R7, R14 to R8, R17 to R9, U13 to U8, Y3 to Y1
Changed lines of the file:
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@@
 		(in_pos_files yes)
 		(dnp no)
-		(property "Reference" "R2"
+		(property "Reference" "R10"
 			(at 175.26 73.025 90)
 			(show_name no)
@@
 			(project "constellation"
 				(path "/ba226b81-7f6b-4f1e-964f-d5311904768c/024ded0e-182d-4822-a380-1069265c1486"
-					(reference "R2")
-					(unit 1)
-				)
-				(path "/ba226b81-7f6b-4f1e-964f-d5311904768c/ee7bb32f-b13d-4ab0-a3c0-7eccf92cdd39"
-					(reference "R3")
+					(reference "R10")
 					(unit 1)
 				)
@@
 		(dnp no)
 		(fields_autoplaced yes)
-		(property "Reference" "U13"
+		(property "Reference" "U8"
 			(at 147.5583 135.255 0)
 			(show_name no)
@@
 			(project "constellation"
 				(path "/ba226b81-7f6b-4f1e-964f-d5311904768c/024ded0e-182d-4822-a380-1069265c1486"
-					(reference "U13")
-					(unit 1)
-				)
-				(path "/ba226b81-7f6b-4f1e-964f-d5311904768c/ee7bb32f-b13d-4ab0-a3c0-7eccf92cdd39"
-					(reference "U14")
+					(reference "U8")
 					(unit 1)
 				)
@@
 		(in_pos_files yes)
 		(dnp no)
-		(property "Reference" "Q4"
+		(property "Reference" "Q2"
 			(at 167.64 70.485 90)
 			(show_name no)
@@
 			(project "constellation"
 				(path "/ba226b81-7f6b-4f1e-964f-d5311904768c/024ded0e-182d-4822-a380-1069265c1486"
-					(reference "Q4")
-					(unit 1)
-				)
-				(path "/ba226b81-7f6b-4f1e-964f-d5311904768c/ee7bb32f-b13d-4ab0-a3c0-7eccf92cdd39"
-					(reference "Q6")
+					(reference "Q2")
 					(unit 1)
 				)
@@
 		(in_pos_files yes)
 		(dnp no)
-		(property "Reference" "C22"
+		(property "Reference" "C12"
 			(at 180.975 79.375 0)
 			(show_name no)
@@
 			(project "constellation"
 				(path "/ba226b81-7f6b-4f1e-964f-d5311904768c/024ded0e-182d-4822-a380-1069265c1486"
-					(reference "C22")
-					(unit 1)
-				)
-				(path "/ba226b81-7f6b-4f1e-964f-d5311904768c/ee7bb32f-b13d-4ab0-a3c0-7eccf92cdd39"
-					(reference "C23")
+					(reference "C12")
 					(unit 1)
 				)
@@
 		(in_pos_files yes)
 		(dnp no)
-		(property "Reference" "#PWR074"
+		(property "Reference" "#PWR036"
 			(at 142.875 80.645 0)
 			(hide yes)
@@
 			(project "constellation"
 				(path "/ba226b81-7f6b-4f1e-964f-d5311904768c/024ded0e-182d-4822-a380-1069265c1486"
-					(reference "#PWR074")
-					(unit 1)
-				)
-				(path "/ba226b81-7f6b-4f1e-964f-d5311904768c/ee7bb32f-b13d-4ab0-a3c0-7eccf92cdd39"
-					(reference "#PWR083")
+					(reference "#PWR036")
 					(unit 1)
 				)
@@
 		(dnp no)
 		(fields_autoplaced yes)
-		(property "Reference" "#PWR081"
+		(property "Reference" "#PWR043"
 			(at 191.77 104.14 0)
 			(hide yes)
@@
 			(project "constellation"
 				(path "/ba226b81-7f6b-4f1e-964f-d5311904768c/024ded0e-182d-4822-a380-1069265c1486"
-					(reference "#PWR081")
-					(unit 1)
-				)
-				(path "/ba226b81-7f6b-4f1e-964f-d5311904768c/ee7bb32f-b13d-4ab0-a3c0-7eccf92cdd39"
-					(reference "#PWR090")
+					(reference "#PWR043")
 					(unit 1)
 				)
@@
 		(dnp no)
 		(fields_autoplaced yes)
-		(property "Reference" "#PWR078"
+		(property "Reference" "#PWR040"
 			(at 166.37 141.605 0)
 			(hide yes)
@@
 			(project "constellation"
 				(path "/ba226b81-7f6b-4f1e-964f-d5311904768c/024ded0e-182d-4822-a380-1069265c1486"
-					(reference "#PWR078")
-					(unit 1)
-				)
-				(path "/ba226b81-7f6b-4f1e-964f-d5311904768c/ee7bb32f-b13d-4ab0-a3c0-7eccf92cdd39"
-					(reference "#PWR087")
+					(reference "#PWR040")
 					(unit 1)
 				)
@@
 		(in_pos_files yes)
 		(dnp no)
-		(property "Reference" "Q3"
+		(property "Reference" "Q1"
 			(at 170.18 91.44 0)
 			(show_name no)
@@
 			(project "constellation"
 				(path "/ba226b81-7f6b-4f1e-964f-d5311904768c/024ded0e-182d-4822-a380-1069265c1486"
-					(reference "Q3")
-					(unit 1)
-				)
-				(path "/ba226b81-7f6b-4f1e-964f-d5311904768c/ee7bb32f-b13d-4ab0-a3c0-7eccf92cdd39"
-					(reference "Q5")
+					(reference "Q1")
 					(unit 1)
 				)
@@
 		(dnp no)
 		(fields_autoplaced yes)
-		(property "Reference" "#PWR075"
+		(property "Reference" "#PWR037"
 			(at 145.415 141.605 0)
 			(hide yes)
@@
 			(project "constellation"
 				(path "/ba226b81-7f6b-4f1e-964f-d5311904768c/024ded0e-182d-4822-a380-1069265c1486"
-					(reference "#PWR075")
-					(unit 1)
-				)
-				(path "/ba226b81-7f6b-4f1e-964f-d5311904768c/ee7bb32f-b13d-4ab0-a3c0-7eccf92cdd39"
-					(reference "#PWR084")
+					(reference "#PWR037")
 					(unit 1)
 				)
@@
 		(dnp no)
 		(fields_autoplaced yes)
-		(property "Reference" "#PWR079"
+		(property "Reference" "#PWR041"
 			(at 167.64 104.14 0)
 			(hide yes)
@@
 			(project "constellation"
 				(path "/ba226b81-7f6b-4f1e-964f-d5311904768c/024ded0e-182d-4822-a380-1069265c1486"
-					(reference "#PWR079")
-					(unit 1)
-				)
-				(path "/ba226b81-7f6b-4f1e-964f-d5311904768c/ee7bb32f-b13d-4ab0-a3c0-7eccf92cdd39"
-					(reference "#PWR088")
+					(reference "#PWR041")
 					(unit 1)
 				)
@@
 		(in_pos_files yes)
 		(dnp no)
-		(property "Reference" "#PWR076"
+		(property "Reference" "#PWR038"
 			(at 160.655 80.645 0)
 			(hide yes)
@@
 			(project "constellation"
 				(path "/ba226b81-7f6b-4f1e-964f-d5311904768c/024ded0e-182d-4822-a380-1069265c1486"
-					(reference "#PWR076")
-					(unit 1)
-				)
-				(path "/ba226b81-7f6b-4f1e-964f-d5311904768c/ee7bb32f-b13d-4ab0-a3c0-7eccf92cdd39"
-					(reference "#PWR085")
+					(reference "#PWR038")
 					(unit 1)
 				)
@@
 		(dnp no)
 		(fields_autoplaced yes)
-		(property "Reference" "#PWR077"
+		(property "Reference" "#PWR039"
 			(at 170.18 125.095 0)
 			(hide yes)
@@
 			(project "constellation"
 				(path "/ba226b81-7f6b-4f1e-964f-d5311904768c/024ded0e-182d-4822-a380-1069265c1486"
-					(reference "#PWR077")
-					(unit 1)
-				)
-				(path "/ba226b81-7f6b-4f1e-964f-d5311904768c/ee7bb32f-b13d-4ab0-a3c0-7eccf92cdd39"
-					(reference "#PWR086")
+					(reference "#PWR039")
 					(unit 1)
 				)
@@
 		(in_pos_files yes)
 		(dnp yes)
-		(property "Reference" "R14"
+		(property "Reference" "R8"
 			(at 167.64 119.3801 0)
 			(show_name no)
@@
 			(project "constellation"
 				(path "/ba226b81-7f6b-4f1e-964f-d5311904768c/024ded0e-182d-4822-a380-1069265c1486"
-					(reference "R14")
-					(unit 1)
-				)
-				(path "/ba226b81-7f6b-4f1e-964f-d5311904768c/ee7bb32f-b13d-4ab0-a3c0-7eccf92cdd39"
-					(reference "R15")
+					(reference "R8")
 					(unit 1)
 				)
@@
 		(in_pos_files yes)
 		(dnp no)
-		(property "Reference" "#PWR080"
+		(property "Reference" "#PWR042"
 			(at 179.07 88.265 0)
 			(hide yes)
@@
 			(project "constellation"
 				(path "/ba226b81-7f6b-4f1e-964f-d5311904768c/024ded0e-182d-4822-a380-1069265c1486"
-					(reference "#PWR080")
-					(unit 1)
-				)
-				(path "/ba226b81-7f6b-4f1e-964f-d5311904768c/ee7bb32f-b13d-4ab0-a3c0-7eccf92cdd39"
-					(reference "#PWR089")
+					(reference "#PWR042")
 					(unit 1)
 				)
@@
 		(in_pos_files yes)
 		(dnp yes)
-		(property "Reference" "R17"
+		(property "Reference" "R9"
 			(at 167.64 130.1751 0)
 			(show_name no)
@@
 			(project "constellation"
 				(path "/ba226b81-7f6b-4f1e-964f-d5311904768c/024ded0e-182d-4822-a380-1069265c1486"
-					(reference "R17")
-					(unit 1)
-				)
-				(path "/ba226b81-7f6b-4f1e-964f-d5311904768c/ee7bb32f-b13d-4ab0-a3c0-7eccf92cdd39"
-					(reference "R19")
+					(reference "R9")
 					(unit 1)
 				)
@@
 		(in_pos_files yes)
 		(dnp no)
-		(property "Reference" "L2"
+		(property "Reference" "L1"
 			(at 182.245 73.025 90)
 			(show_name no)
@@
 			(project "constellation"
 				(path "/ba226b81-7f6b-4f1e-964f-d5311904768c/024ded0e-182d-4822-a380-1069265c1486"
-					(reference "L2")
-					(unit 1)
-				)
-				(path "/ba226b81-7f6b-4f1e-964f-d5311904768c/ee7bb32f-b13d-4ab0-a3c0-7eccf92cdd39"
-					(reference "L3")
+					(reference "L1")
 					(unit 1)
 				)
@@
 		(in_pos_files yes)
 		(dnp no)
-		(property "Reference" "J2"
+		(property "Reference" "J1"
 			(at 194.31 85.725 0)
 			(show_name no)
@@
 			(project "constellation"
 				(path "/ba226b81-7f6b-4f1e-964f-d5311904768c/024ded0e-182d-4822-a380-1069265c1486"
-					(reference "J2")
-					(unit 1)
-				)
-				(path "/ba226b81-7f6b-4f1e-964f-d5311904768c/ee7bb32f-b13d-4ab0-a3c0-7eccf92cdd39"
-					(reference "J3")
+					(reference "J1")
 					(unit 1)
 				)
@@
 		(in_pos_files yes)
 		(dnp no)
-		(property "Reference" "#PWR073"
+		(property "Reference" "#PWR035"
 			(at 140.335 80.645 0)
 			(hide yes)
@@
 			(project "constellation"
 				(path "/ba226b81-7f6b-4f1e-964f-d5311904768c/024ded0e-182d-4822-a380-1069265c1486"
-					(reference "#PWR073")
-					(unit 1)
-				)
-				(path "/ba226b81-7f6b-4f1e-964f-d5311904768c/ee7bb32f-b13d-4ab0-a3c0-7eccf92cdd39"
-					(reference "#PWR082")
+					(reference "#PWR035")
 					(unit 1)
 				)
@@
 		(in_pos_files yes)
 		(dnp no)
-		(property "Reference" "R16"
+		(property "Reference" "R7"
 			(at 161.925 79.3751 0)
 			(show_name no)
@@
 			(project "constellation"
 				(path "/ba226b81-7f6b-4f1e-964f-d5311904768c/024ded0e-182d-4822-a380-1069265c1486"
-					(reference "R16")
-					(unit 1)
-				)
-				(path "/ba226b81-7f6b-4f1e-964f-d5311904768c/ee7bb32f-b13d-4ab0-a3c0-7eccf92cdd39"
-					(reference "R18")
+					(reference "R7")
 					(unit 1)
 				)
@@
 		(in_pos_files yes)
 		(dnp no)
-		(property "Reference" "Y3"
+		(property "Reference" "Y1"
 			(at 119.38 125.0949 90)
 			(show_name no)
@@
 			(project "constellation"
 				(path "/ba226b81-7f6b-4f1e-964f-d5311904768c/024ded0e-182d-4822-a380-1069265c1486"
-					(reference "Y3")
-					(unit 1)
-				)
-				(path "/ba226b81-7f6b-4f1e-964f-d5311904768c/ee7bb32f-b13d-4ab0-a3c0-7eccf92cdd39"
-					(reference "Y4")
-					(unit 1)
-				)
+					(reference "Y1")
+					(unit 1)
+				)
