File: Hardware/constellation/accelerometer.kicad_sch (KiCad schematic)
At the start: 4 parts, among them U7 H3LIS331DL

Commit message: add the hierarchal pins to the imu block
Connections:
- net H3L_INT2 is gone; now on net H3L_INT1: U7.9 (INT2)
Changed lines of the file:
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@@
 		)
 	)
-	(global_label "H3L_SCK"
+	(hierarchical_label "H3L_CS"
 		(shape input)
-		(at 120.015 100.33 180)
-		(fields_autoplaced yes)
+		(at 120.015 97.79 180)
 		(effects
 			(font
@@
 			(justify right)
 		)
-		(property "Intersheetrefs" "${INTERSHEET_REFS}"
-			(at 101.0037 100.33 0)
-			(hide yes)
-			(show_name no)
-			(do_not_autoplace no)
-			(effects
-				(font
-					(size 1.27 1.27)
-				)
-				(justify right)
-			)
-		)
 	)
-	(global_label "H3L_INT1"
+	(hierarchical_label "H3L_INT1"
 		(shape input)
-		(at 161.925 100.33 0)
-		(fields_autoplaced yes)
+		(at 161.925 102.87 0)
 		(effects
 			(font
@@
 			(justify left)
 		)
-		(property "Intersheetrefs" "${INTERSHEET_REFS}"
-			(at 180.9363 100.33 0)
-			(hide yes)
-			(show_name no)
-			(do_not_autoplace no)
-			(effects
-				(font
-					(size 1.27 1.27)
-				)
-				(justify left)
-			)
-		)
 	)
-	(global_label "H3L_MOSI"
+	(hierarchical_label "H3L_MISO"
 		(shape input)
-		(at 120.015 105.41 180)
-		(fields_autoplaced yes)
+		(at 120.015 102.87 180)
 		(effects
 			(font
@@
 			(justify right)
 		)
-		(property "Intersheetrefs" "${INTERSHEET_REFS}"
-			(at 101.0037 105.41 0)
-			(hide yes)
-			(show_name no)
-			(do_not_autoplace no)
-			(effects
-				(font
-					(size 1.27 1.27)
-				)
-				(justify right)
+	)
+	(hierarchical_label "H3L_INT1"
+		(shape input)
+		(at 161.925 100.33 0)
+		(effects
+			(font
+				(size 1.27 1.27)
 			)
+			(justify left)
 		)
 	)
-	(global_label "H3L_MISO"
+	(hierarchical_label "H3L_MOSI"
 		(shape input)
-		(at 120.015 102.87 180)
-		(fields_autoplaced yes)
+		(at 120.015 105.41 180)
 		(effects
 			(font
@@
 			(justify right)
 		)
-		(property "Intersheetrefs" "${INTERSHEET_REFS}"
-			(at 101.0037 102.87 0)
-			(hide yes)
-			(show_name no)
-			(do_not_autoplace no)
-			(effects
-				(font
-					(size 1.27 1.27)
-				)
-				(justify right)
-			)
-		)
 	)
-	(global_label "H3L_INT2"
+	(hierarchical_label "H3L_SCK"
 		(shape input)
-		(at 161.925 102.87 0)
-		(fields_autoplaced yes)
-		(effects
-			(font
-				(size 1.27 1.27)
-			)
-			(justify left)
-		)
-		(property "Intersheetrefs" "${INTERSHEET_REFS}"
-			(at 180.9363 102.87 0)
-			(hide yes)
-			(show_name no)
-			(do_not_autoplace no)
-			(effects
-				(font
-					(size 1.27 1.27)
-				)
-				(justify left)
-			)
-		)
-	)
-	(global_label "H3L_CS"
-		(shape input)
-		(at 120.015 97.79 180)
-		(fields_autoplaced yes)
+		(at 120.015 100.33 180)
 		(effects
 			(font
@@
 			(justify right)
 		)
-		(property "Intersheetrefs" "${INTERSHEET_REFS}"
-			(at 101.0037 97.79 0)
-			(hide yes)
-			(show_name no)
-			(do_not_autoplace no)
-			(effects
-				(font
-					(size 1.27 1.27)
-				)
-				(justify right)
-			)
-		)
 	)

Commit message: add gnss short detection and lna_en supervisor
Connections:
- net H3L_INT1: no longer U7.9 (INT2)
- new net H3L_INT2: U7.9 (INT2)
Changed lines of the file:
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@@
 		)
 	)
-	(hierarchical_label "H3L_INT1"
+	(hierarchical_label "H3L_INT2"
 		(shape input)
 		(at 161.925 102.87 0)

Commit message: add lr2021 footprint and comms
Parts:
- renumbered C8 to C10
Changed lines of the file:
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@@
 		(dnp no)
 		(fields_autoplaced yes)
-		(property "Reference" "#PWR026"
+		(property "Reference" "#PWR031"
 			(at 150.495 121.92 0)
 			(hide yes)
@@
 			(project "constellation"
 				(path "/ba226b81-7f6b-4f1e-964f-d5311904768c/8ef0bafe-e56b-4ed3-8e19-af101ba69e51"
-					(reference "#PWR026")
+					(reference "#PWR031")
 					(unit 1)
 				)
@@
 		(dnp no)
 		(fields_autoplaced yes)
-		(property "Reference" "#PWR029"
+		(property "Reference" "#PWR033"
 			(at 167.005 90.805 0)
 			(hide yes)
@@
 			(project "constellation"
 				(path "/ba226b81-7f6b-4f1e-964f-d5311904768c/8ef0bafe-e56b-4ed3-8e19-af101ba69e51"
-					(reference "#PWR029")
+					(reference "#PWR033")
 					(unit 1)
 				)
@@
 		(dnp no)
 		(fields_autoplaced yes)
-		(property "Reference" "#PWR028"
+		(property "Reference" "#PWR030"
 			(at 130.81 90.805 0)
 			(hide yes)
@@
 			(project "constellation"
 				(path "/ba226b81-7f6b-4f1e-964f-d5311904768c/8ef0bafe-e56b-4ed3-8e19-af101ba69e51"
-					(reference "#PWR028")
+					(reference "#PWR030")
 					(unit 1)
 				)
@@
 		(in_pos_files yes)
 		(dnp no)
-		(property "Reference" "#PWR027"
+		(property "Reference" "#PWR032"
 			(at 151.765 90.805 0)
 			(hide yes)
@@
 			(project "constellation"
 				(path "/ba226b81-7f6b-4f1e-964f-d5311904768c/8ef0bafe-e56b-4ed3-8e19-af101ba69e51"
-					(reference "#PWR027")
+					(reference "#PWR032")
 					(unit 1)
 				)
@@
 		(dnp no)
 		(fields_autoplaced yes)
-		(property "Reference" "#PWR030"
+		(property "Reference" "#PWR034"
 			(at 175.895 103.505 0)
 			(hide yes)
@@
 			(project "constellation"
 				(path "/ba226b81-7f6b-4f1e-964f-d5311904768c/8ef0bafe-e56b-4ed3-8e19-af101ba69e51"
-					(reference "#PWR030")
+					(reference "#PWR034")
 					(unit 1)
 				)
@@
 		(in_pos_files yes)
 		(dnp no)
-		(property "Reference" "C8"
+		(property "Reference" "C10"
 			(at 168.91 91.44 0)
 			(show_name no)
@@
 			(project "constellation"
 				(path "/ba226b81-7f6b-4f1e-964f-d5311904768c/8ef0bafe-e56b-4ed3-8e19-af101ba69e51"
-					(reference "C8")
-					(unit 1)
-				)
+					(reference "C10")
+					(unit 1)
+				)

Commit message: add pyro stuff, start system power
Changed lines of the file:
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@@
 	)
 	(hierarchical_label "H3L_INT2"
-		(shape input)
+		(shape output)
 		(at 161.925 102.87 0)
 		(effects
@@
 	)
 	(hierarchical_label "H3L_MISO"
-		(shape input)
+		(shape output)
 		(at 120.015 102.87 180)
 		(effects
@@
 	)
 	(hierarchical_label "H3L_INT1"
-		(shape input)
+		(shape output)
 		(at 161.925 100.33 0)
 		(effects
