File: Hardware/constellation/lora.kicad_sch (KiCad schematic)
At the start: 0 parts

Commit message: add lr2021 footprint and comms
Parts:
- added L2: 2.2uH, Inductor_SMD:L_0603_1608Metric, symbol Device:L_Small
- added R11: 10K, Resistor_SMD:R_0402_1005Metric_Pad0.72x0.64mm_HandSolder, symbol Device:R_Small
- added R12, R13, R14, R15, R16, R17: 470, Resistor_SMD:R_0402_1005Metric, symbol Device:R_Small
- added U9: LR2021, symbol LR2021:LR2021
Connections:
- new net: R15.2, U9.22 (MOSI)
- new net: R14.2, U9.21 (MISO)
- new net: R16.2, U9.25 (BUSY)
- new net: R17.2, U9.24 (NRESET)
- new net: R13.2, U9.23 (SCK)
- new net: R11.2, R12.2, U9.24 (NRESET)
- new net: L2.1, U9.16 (LXA)
- new net: L2.2, U9.14 (LXB)
- new net GND: U9.0 (GND), U9.15 (GND), U9.30 (GND)
- new net LR2021_BUSY: R16.1
- new net LR2021_CS: R12.1
- new net LR2021_MISO: R14.1
- new net LR2021_MOSI: R15.1
- new net LR2021_NRESET: R17.1
- new net LR2021_SCK: R13.1
- new net VDD: R11.1

Commit message: finish LORA sheet
Parts:
- removed U9: LR2021, symbol LR2021:LR2021
- added C13: 47pF, Capacitor_SMD:C_0402_1005Metric, symbol Device:C_Small
- added C14: 47nF, Capacitor_SMD:C_0402_1005Metric, symbol Device:C_Small
- added C15: 470nF, Capacitor_SMD:C_0402_1005Metric, symbol Device:C_Small
- added C16, C20: 100nF, Capacitor_SMD:C_0402_1005Metric, symbol Device:C_Small
- added C17, C21: 1uF, Capacitor_SMD:C_0402_1005Metric, symbol Device:C_Small
- added C18: 1nF, Capacitor_SMD:C_0402_1005Metric, symbol Device:C_Small
- added C19: 10pF, Capacitor_SMD:C_0402_1005Metric, symbol Device:C_Small
- added FL1: 0900FM15K0039, RF_Converter:Balun_Johanson_0900FM15K0039, symbol Filter:0900FM15K0039
- added J2: Conn_Coaxial, Connector_Coaxial:SMA_Amphenol_132291-12_Vertical, symbol Connector:Conn_Coaxial
- added L3: 15uH, Inductor_SMD:L_0402_1005Metric, symbol Device:L_Small
- added R18: 100, Resistor_SMD:R_0402_1005Metric, symbol Device:R_Small
- added R19: 220, Resistor_SMD:R_0402_1005Metric, symbol Device:R_Small
- added U10: PE4259, Package_TO_SOT_SMD:SOT-363_SC-70-6, symbol 2025-12-25_01-02-53:PE4259
- added U9: SX1262IMLTRT, Package_DFN_QFN:QFN-24-1EP_4x4mm_P0.5mm_EP2.6x2.6mm, symbol RF:SX1262IMLTRT
- added Y2: NT2016SA-32M-END4263A, Oscillator:Oscillator_SMD_SeikoEpson_TG2520SMN-xxx-xxxxxx-4Pin_2.5x2.0mm, symbol Oscillator:TG2520SMN-xx.xxxxxxMhz-xxxxNM
- L2: value 2.2uH -> 47nH; footprint Inductor_SMD:L_0603_1608Metric -> Inductor_SMD:L_0402_1005Metric
Connections:
- net GND: now also C13.2, C14.2, C15.2, C16.2, C17.2, C18.2, C20.2, C21.2, FL1.10 (GND), FL1.2 (GND), FL1.5 (GND), FL1.7 (GND), FL1.9 (GND), J2.2 (Ext), U10.2 (GND), U9.2 (GND), U9.20 (GND), U9.25 (GND), U9.5 (GND), U9.8 (GND), Y2.2 (GND)
- net VDD: now also C16.1, C17.1, C21.1, U10.6 (VDD), U9.1 (VDD_IN), U9.10 (VBAT), U9.11 (VBAT_IO)
- net at R15.2: now also U9.17 (MOSI)
- net at R14.2: now also U9.16 (MISO)
- net at R16.2: now also U9.14 (BUSY)
- net at R17.2: now also U9.15 (~{RESET})
- net at R13.2: now also U9.18 (SCK)
- net at R11.2, R12.2: now also U9.19 (NSS)
- net at L2.1: now also C13.1, C14.1, U9.24 (VR_PA)
- net at L2.2: now also FL1.1 (RFO), U9.23 (RFO)
- new net: R19.1, Y2.3 (OUT)
- new net: C20.1, U9.6 (DIO3), Y2.4 (Vcc)
- new net: J2.1 (In), U10.5 (RFIN)
- new net: FL1.4 (RFI_P), U9.21 (RFI_P)
- new net: FL1.3 (RFI_N), U9.22 (RFI_N)
- new net: C19.2, U9.3 (XTA)
- new net: C15.1, L3.1, U9.7 (VREG)
- new net: L3.2, U9.9 (DCC_SW)
- new net: C19.1, R19.2
- new net: FL1.6 (SW_RFI), U10.3 (RF2)
- new net: FL1.8 (SW_RFO), U10.1 (RF1)
- new net: C18.1, R18.1, U10.4 (CTRL)
- new net ANT_SW: R18.2, U9.12 (DIO2)
- new net LR2021_IRQ: U9.13 (DIO1)
- no-connect marks 0 -> 1
Other:
- moved on the sheet: R11, R12, R13, R14, R15, R16, R17

Commit message: add pyro stuff, start system power
Parts:
- Y2: footprint Oscillator:Oscillator_SMD_SeikoEpson_TG2520SMN-xxx-xxxxxx-4Pin_2.5x2.0mm -> Oscillator:Oscillator_SMD_SiT_PQFN-4Pin_2.0x1.6mm
Connections:
- net LR2021_BUSY renamed SX1262_BUSY
- net LR2021_CS renamed SX1262_CS
- net LR2021_IRQ renamed SX1262_IRQ
- net LR2021_MISO renamed SX1262_MISO
- net LR2021_MOSI renamed SX1262_MOSI
- net LR2021_NRESET renamed SX1262_NRESET
- net LR2021_SCK renamed SX1262_SCK
Other:
- moved on the sheet: C13, C14, C15, C16, C17, C18, C19, C20, C21, FL1, J2, L2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
