File: Hardware/constellation/magnetometer.kicad_sch (KiCad schematic)
At the start: 4 parts, among them U6 MMC5983MA

Commit message: add pyro stuff, start system power
Changed lines of the file:
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@@
 	)
 	(hierarchical_label "MMC_INT"
-		(shape input)
+		(shape output)
 		(at 161.29 95.25 0)
 		(effects
@@
 	)
 	(hierarchical_label "MMC_MISO"
-		(shape input)
+		(shape output)
 		(at 111.76 100.33 180)
 		(effects
